File: pmic.kicad_sch (KiCad schematic)
At the start: 12 parts, among them SW2 PWR_BTN, U1 NPM1300-CAAA-R

Commit message: fixed ERC warnings, finalized PMIC
Parts:
- added J3: Battery Connector, symbol Connector:Conn_01x02_Pin
- U1: footprint NPM1300-CAAA-R:BGA35N44X41P5X7_237X307X51 -> TheSummitProject:BGA35N44X41P5X7_237X307X51
Connections:
- net +BATT renamed VBAT
- net VBAT: now also J3.1 (Pin_1)
- net -BATT renamed GND
- net GND: now also J3.2 (Pin_2)
Other:
- note added: "Battery Pins"
- moved on the sheet: C20, C21, C22, D1, L1, L2, R2, R3, R4, SW2, TH1, U1

Commit message: added symbol library
Parts:
- U1: symbol STM32U5F7VJT6:NPM1300-CAAA-R -> TheSummitProject:NPM1300-CAAA-R
Changed lines of the file:
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@@
+	)
+	(junction
+		(at 185.42 135.89)
+		(diameter 0)
+		(color 0 0 0 0)
 	)
 	(junction
@@
 	)
 	(junction
+		(at 187.96 135.89)
+		(diameter 0)
+		(color 0 0 0 0)
+	)
+	(junction
 		(at 73.66 49.53)
 		(diameter 0)
@@
 		(color 0 0 0 0)
 	)
-	(junction
-		(at 182.88 135.89)
-		(diameter 0)
-		(color 0 0 0 0)
-	)
 	(no_connect
 		(at 182.88 90.17)
@@
 	(wire
 		(pts
+			(xy 182.88 133.35) (xy 187.96 133.35)
+		)
+		(stroke
+			(width 0)
+			(type default)
+		)
+	)
+	(wire
+		(pts
 			(xy 127 87.63) (xy 127 88.9)
 		)
@@
 	(wire
 		(pts
-			(xy 182.88 135.89) (xy 186.69 135.89)
-		)
-		(stroke
-			(width 0)
-			(type default)
-		)
-	)
-	(wire
-		(pts
 			(xy 219.71 119.38) (xy 219.71 97.79)
 		)
@@
 	(wire
 		(pts
+			(xy 182.88 135.89) (xy 185.42 135.89)
+		)
+		(stroke
+			(width 0)
+			(type default)
+		)
+	)
+	(wire
+		(pts
 			(xy 198.12 107.95) (xy 198.12 110.49)
 		)
@@
 	(wire
 		(pts
-			(xy 182.88 133.35) (xy 182.88 135.89)
+			(xy 190.5 135.89) (xy 187.96 135.89)
 		)
 		(stroke
@@
 	(wire
 		(pts
-			(xy 182.88 135.89) (xy 182.88 138.43)
+			(xy 182.88 138.43) (xy 185.42 138.43)
 		)
 		(stroke
@@
 	(wire
 		(pts
+			(xy 187.96 133.35) (xy 187.96 135.89)
+		)
+		(stroke
+			(width 0)
+			(type default)
+		)
+	)
+	(wire
+		(pts
 			(xy 182.88 120.65) (xy 189.23 120.65)
 		)
@@
 	(wire
 		(pts
+			(xy 185.42 135.89) (xy 187.96 135.89)
+		)
+		(stroke
+			(width 0)
+			(type default)
+		)
+	)
+	(wire
+		(pts
 			(xy 120.65 102.87) (xy 127 102.87)
+		)
+		(stroke
+			(width 0)
+			(type default)
+		)
+	)
+	(wire
+		(pts
+			(xy 185.42 138.43) (xy 185.42 135.89)
 		)
 		(stroke
@@
 	(symbol
 		(lib_id "power:GND")
-		(at 186.69 135.89 90)
+		(at 190.5 135.89 90)
 		(unit 1)
 		(body_style 1)
@@
 		(fields_autoplaced yes)
 		(property "Reference" "#PWR046"
-			(at 193.04 135.89 0)
+			(at 196.85 135.89 0)
 			(hide yes)
 			(show_name no)
@@
 		)
 		(property "Value" "GND"
-			(at 190.5 135.8899 90)
+			(at 194.31 135.8899 90)
 			(show_name no)
 			(do_not_autoplace no)
@@
 		)
 		(property "Footprint" ""
-			(at 186.69 135.89 0)
+			(at 190.5 135.89 0)
 			(hide yes)
 			(show_name no)
@@
 		)
 		(property "Datasheet" ""
-			(at 186.69 135.89 0)
+			(at 190.5 135.89 0)
 			(hide yes)
 			(show_name no)
@@
 		)
 		(property "Description" "Power symbol creates a global label with name \"GND\" , ground"
-			(at 186.69 135.89 0)
+			(at 190.5 135.89 0)
 			(hide yes)
 			(show_name no)
@@
 	)
 	(symbol
-		(lib_id "STM32U5F7VJT6:NPM1300-CAAA-R")
+		(lib_id "TheSummitProject:NPM1300-CAAA-R")
 		(at 154.94 105.41 0)
 		(unit 1)
