File: peripherals.kicad_sch (KiCad schematic)
At the start: 25 parts, among them J2 GPS_ANT, U5 BME280, U6 LSM303AGR, U7 MAX-M10S-00B, U8 RAK4630, U9 SN74AVC2T245RSWR

Commit message: Changed SPI to 3-wire, added Accelerometer interupt
Connections:
- net GPS_RX: now also U7.2 (TXD); no longer U7.3 (RXD)
- net GPS_TX: now also U7.3 (RXD); no longer U7.2 (TXD)
- net ACC_INT: now reaches U6.12 (INT_1_XL)
- net SNSR_MISO: no longer names the net of U5.5 (SDO)
Other:
- note removed: "FALLING DETECT, CONNECT INTERRUPT"
- moved on the sheet: C38
Changed lines of the file:
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@@
 		)
 	)
-	(text "FALLING DETECT, CONNECT INTERRUPT"
-		(exclude_from_sim no)
-		(at 77.978 165.862 0)
-		(effects
-			(font
-				(size 1.27 1.27)
-			)
-		)
-	)
 	(text "LoRa\n"
 		(exclude_from_sim no)
@@
 	)
 	(junction
-		(at 93.98 55.88)
+		(at 96.52 124.46)
 		(diameter 0)
 		(color 0 0 0 0)
 	)
 	(junction
-		(at 234.95 36.83)
+		(at 93.98 55.88)
 		(diameter 0)
 		(color 0 0 0 0)
 	)
 	(junction
-		(at 252.73 132.08)
+		(at 234.95 36.83)
 		(diameter 0)
 		(color 0 0 0 0)
 	)
 	(junction
-		(at 234.95 34.29)
+		(at 252.73 132.08)
 		(diameter 0)
 		(color 0 0 0 0)
 	)
 	(junction
-		(at 96.52 127)
+		(at 234.95 34.29)
 		(diameter 0)
 		(color 0 0 0 0)
@@
 	)
 	(junction
-		(at 96.52 124.46)
+		(at 189.23 41.91)
 		(diameter 0)
 		(color 0 0 0 0)
 	)
 	(junction
-		(at 189.23 41.91)
+		(at 105.41 127)
 		(diameter 0)
 		(color 0 0 0 0)
@@
 	)
 	(no_connect
-		(at 87.63 132.08)
-	)
-	(no_connect
 		(at 237.49 69.85)
 	)
@@
 	)
 	(no_connect
+		(at 149.86 44.45)
+	)
+	(no_connect
 		(at 240.03 128.27)
 	)
@@
 	(wire
 		(pts
-			(xy 96.52 124.46) (xy 104.14 124.46)
-		)
-		(stroke
-			(width 0)
-			(type default)
-		)
-	)
-	(wire
-		(pts
-			(xy 87.63 127) (xy 96.52 127)
+			(xy 96.52 124.46) (xy 101.6 124.46)
 		)
 		(stroke
@@
 	(wire
 		(pts
+			(xy 87.63 127) (xy 105.41 127)
+		)
+		(stroke
+			(width 0)
+			(type default)
+		)
+	)
+	(wire
+		(pts
 			(xy 137.16 33.02) (xy 137.16 36.83)
 		)
@@
 	(wire
 		(pts
-			(xy 96.52 127) (xy 104.14 127)
+			(xy 105.41 127) (xy 115.57 127)
 		)
 		(stroke
@@
 		)
 	)
+	(global_label "ACC_INT"
+		(shape input)
+		(at 87.63 132.08 0)
+		(fields_autoplaced yes)
+		(effects
+			(font
+				(size 1.27 1.27)
+			)
+			(justify left)
+		)
+		(property "Intersheetrefs" "${INTERSHEET_REFS}"
+			(at 98.1143 132.08 0)
+			(hide yes)
+			(show_name no)
+			(do_not_autoplace no)
+			(effects
+				(font
+					(size 1.27 1.27)
+				)
+				(justify left)
+			)
+		)
+	)
 	(global_label "LoRA-"
 		(shape input)
@@
 	(global_label "GPS_TX"
 		(shape input)
-		(at 81.28 71.12 0)
+		(at 81.28 73.66 0)
 		(fields_autoplaced yes)
 		(effects
@@
 		)
 		(property "Intersheetrefs" "${INTERSHEET_REFS}"
-			(at 91.1594 71.12 0)
+			(at 91.1594 73.66 0)
 			(hide yes)
 			(show_name no)
@@
 		)
 	)
-	(global_label "GPS_RX"
-		(shape input)
-		(at 81.28 73.66 0)
-		(fields_autoplaced yes)
-		(effects
-			(font
-				(size 1.27 1.27)
-			)
-			(justify left)
-		)
-		(property "Intersheetrefs" "${INTERSHEET_REFS}"
-			(at 91.4618 73.66 0)
-			(hide yes)
-			(show_name no)
-			(do_not_autoplace no)
-			(effects
-				(font
-					(size 1.27 1.27)
-				)
-				(justify left)
-			)
-		)
-	)
-	(global_label "SNSR_MISO"
-		(shape input)
-		(at 149.86 44.45 0)
-		(fields_autoplaced yes)
-		(effects
-			(font
-				(size 1.27 1.27)
-			)
-			(justify left)
-		)
-		(property "Intersheetrefs" "${INTERSHEET_REFS}"
-			(at 163.4285 44.45 0)
-			(hide yes)
-			(show_name no)
-			(do_not_autoplace no)
-			(effects
-				(font
-					(size 1.27 1.27)
-				)
-				(justify left)
-			)
-		)
-	)
 	(global_label "NRF_RST"
 		(shape input)
@@
 		)
 	)
+	(global_label "GPS_RX"
+		(shape input)
+		(at 81.28 71.12 0)
+		(fields_autoplaced yes)
+		(effects
+			(font
+				(size 1.27 1.27)
+			)
+			(justify left)
+		)
+		(property "Intersheetrefs" "${INTERSHEET_REFS}"
+			(at 91.4618 71.12 0)
+			(hide yes)
+			(show_name no)
+			(do_not_autoplace no)
+			(effects
+				(font
+					(size 1.27 1.27)
+				)
+				(justify left)
+			)
+		)
+	)
 	(global_label "LoRa_TX"
 		(shape input)
@@
 	(symbol
 		(lib_id "Device:C")
-		(at 96.52 130.81 0)
+		(at 105.41 130.81 0)
 		(unit 1)
 		(body_style 1)
@@
 		(fields_autoplaced yes)
 		(property "Reference" "C38"
-			(at 100.33 129.5399 0)
+			(at 109.22 129.5399 0)
 			(show_name no)
 			(do_not_autoplace no)
@@
 		)
 		(property "Value" "100n"
-			(at 100.33 132.0799 0)
+			(at 109.22 132.0799 0)
 			(show_name no)
 			(do_not_autoplace no)
@@
 		)
 		(property "Footprint" "Capacitor_SMD:C_0603_1608Metric"
-			(at 97.4852 134.62 0)
+			(at 106.3752 134.62 0)
 			(hide yes)
 			(show_name no)
@@
 		)
 		(property "Datasheet" ""
-			(at 96.52 130.81 0)
+			(at 105.41 130.81 0)
 			(hide yes)
 			(show_name no)
@@
 		)
 		(property "Description" "Unpolarized capacitor"
-			(at 96.52 130.81 0)
+			(at 105.41 130.81 0)
 			(hide yes)
 			(show_name no)
@@
 	(symbol
 		(lib_id "power:+1V8")
-		(at 104.14 124.46 270)
+		(at 101.6 124.46 270)
 		(unit 1)
 		(body_style 1)
@@
 		(in_pos_files yes)
 		(dnp no)
-		(fields_autoplaced yes)
 		(property "Reference" "#PWR0111"
-			(at 100.33 124.46 0)
+			(at 97.79 124.46 0)
 			(hide yes)
 			(show_name no)
@@
 		)
 		(property "Value" "+1.8V"
-			(at 107.95 124.4599 90)
+			(at 104.902 124.46 90)
 			(show_name no)
 			(do_not_autoplace no)
@@
 		)
 		(property "Footprint" ""
-			(at 104.14 124.46 0)
+			(at 101.6 124.46 0)
 			(hide yes)
 			(show_name no)
@@
 		)
 		(property "Datasheet" ""
-			(at 104.14 124.46 0)
+			(at 101.6 124.46 0)
 			(hide yes)
 			(show_name no)
@@
 		)
 		(property "Description" "Power symbol creates a global label with name \"+1V8\""
-			(at 104.14 124.46 0)
+			(at 101.6 124.46 0)
 			(hide yes)
 			(show_name no)
@@
 	(symbol
 		(lib_id "power:+1V8")
-		(at 104.14 127 270)
+		(at 115.57 127 0)
 		(unit 1)
 		(body_style 1)
@@
 		(in_pos_files yes)
 		(dnp no)
-		(fields_autoplaced yes)
 		(property "Reference" "#PWR082"
-			(at 100.33 127 0)
+			(at 115.57 130.81 0)
 			(hide yes)
 			(show_name no)
@@
 		)
 		(property "Value" "+1.8V"
-			(at 107.95 126.9999 90)
+			(at 112.268 122.682 0)
 			(show_name no)
 			(do_not_autoplace no)
@@
 		)
 		(property "Footprint" ""
-			(at 104.14 127 0)
+			(at 115.57 127 0)
 			(hide yes)
 			(show_name no)
@@
 		)
 		(property "Datasheet" ""
-			(at 104.14 127 0)
+			(at 115.57 127 0)
 			(hide yes)
 			(show_name no)
@@
 		)
 		(property "Description" "Power symbol creates a global label with name \"+1V8\""
-			(at 104.14 127 0)
+			(at 115.57 127 0)
 			(hide yes)
 			(show_name no)
@@
 	(symbol
 		(lib_id "power:GND")
-		(at 96.52 134.62 0)
+		(at 105.41 134.62 0)
 		(unit 1)
 		(body_style 1)
@@
 		(fields_autoplaced yes)
 		(property "Reference" "#PWR085"
-			(at 96.52 140.97 0)
+			(at 105.41 140.97 0)
 			(hide yes)
 			(show_name no)
@@
 		)
 		(property "Value" "GND"
-			(at 96.52 139.7 0)
+			(at 105.41 139.7 0)
 			(show_name no)
 			(do_not_autoplace no)
@@
 		)
 		(property "Footprint" ""
-			(at 96.52 134.62 0)
+			(at 105.41 134.62 0)
 			(hide yes)
 			(show_name no)
@@
 		)
 		(property "Datasheet" ""
-			(at 96.52 134.62 0)
+			(at 105.41 134.62 0)
 			(hide yes)
 			(show_name no)
@@
 		)
 		(property "Description" "Power symbol creates a global label with name \"GND\" , ground"
-			(at 96.52 134.62 0)
+			(at 105.41 134.62 0)
 			(hide yes)
 			(show_name no)

Commit message: pcb draft, cleaned up schematic
Parts:
- added BZ1: PKLCS1212E4001-R1, Buzzer_Beeper:Buzzer_Murata_PKLCS1212E, symbol Device:Buzzer
- added R29: 100, Resistor_SMD:R_0603_1608Metric, symbol Device:R
Connections:
- new net: BZ1.2 (-), R29.2
- new net PIEZO_P1: BZ1.1 (+)
- new net PIEZO_P2: R29.1
Other:
- note added: "Buzzer"
