File: screen.kicad_sch (KiCad schematic)
At the start: 11 parts, among them J4 Screen FPC, Q1 NMOS

Commit message: assigned footprint and created PCB file
Parts:
- C25, C26, C27: footprint (none) -> Capacitor_SMD:C_0603_1608Metric
- J4: footprint (none) -> Connector_PinHeader_2.54mm:PinHeader_1x40_P2.54mm_Vertical
- Q1: footprint (none) -> Package_TO_SOT_SMD:SOT-23
- R10, R11, R6, R7, R8, R9: footprint (none) -> Resistor_SMD:R_0603_1608Metric
Changed lines of the file:
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@@
 			)
 		)
-		(property "Footprint" ""
+		(property "Footprint" "Package_TO_SOT_SMD:SOT-23"
 			(at 193.04 93.98 0)
 			(hide yes)
@@
 			)
 		)
-		(property "Footprint" ""
+		(property "Footprint" "Resistor_SMD:R_0603_1608Metric"
 			(at 178.562 102.87 90)
 			(hide yes)
@@
 			)
 		)
-		(property "Footprint" ""
+		(property "Footprint" "Resistor_SMD:R_0603_1608Metric"
 			(at 183.642 85.09 90)
 			(hide yes)
@@
 			)
 		)
-		(property "Footprint" ""
+		(property "Footprint" "Resistor_SMD:R_0603_1608Metric"
 			(at 173.99 94.742 90)
 			(hide yes)
@@
 			)
 		)
-		(property "Footprint" ""
+		(property "Footprint" "Connector_PinHeader_2.54mm:PinHeader_1x40_P2.54mm_Vertical"
 			(at 148.59 66.04 0)
 			(hide yes)
@@
 			)
 		)
-		(property "Footprint" ""
+		(property "Footprint" "Resistor_SMD:R_0603_1608Metric"
 			(at 104.14 97.028 90)
 			(hide yes)
@@
 			)
 		)
-		(property "Footprint" ""
+		(property "Footprint" "Resistor_SMD:R_0603_1608Metric"
 			(at 104.14 86.868 90)
 			(hide yes)
@@
 			)
 		)
-		(property "Footprint" ""
+		(property "Footprint" "Capacitor_SMD:C_0603_1608Metric"
 			(at 123.19 136.1948 0)
 			(hide yes)
@@
 			)
 		)
-		(property "Footprint" ""
+		(property "Footprint" "Resistor_SMD:R_0603_1608Metric"
 			(at 104.14 107.188 90)
 			(hide yes)
@@
 			)
 		)
-		(property "Footprint" ""
+		(property "Footprint" "Capacitor_SMD:C_0603_1608Metric"
 			(at 111.76 119.6848 0)
 			(hide yes)
@@
 			)
 		)
-		(property "Footprint" ""
+		(property "Footprint" "Capacitor_SMD:C_0603_1608Metric"
 			(at 123.19 123.4948 0)
 			(hide yes)

Commit message: migrated display power with lora
Connections:
- net +3.3V_DISP is gone; now on net +3.3V_DP_LORA: J4.33 (Pin_33)
- net +3.3V renamed +3.3V_DP_LORA
Changed lines of the file:
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@@
 			)
 		)
-		(property "Value" "+3.3V"
-			(at 196.85 80.518 0)
+		(property "Value" "+3.3V_DP_LORA"
+			(at 202.184 80.518 0)
 			(show_name no)
 			(do_not_autoplace no)
@@
 		(in_pos_files yes)
 		(dnp no)
-		(fields_autoplaced yes)
 		(property "Reference" "#PWR054"
 			(at 115.57 133.35 0)
@@
 			)
 		)
-		(property "Value" "+3.3V"
-			(at 115.57 142.24 0)
-			(show_name no)
-			(do_not_autoplace no)
-			(effects
-				(font
-					(size 1.27 1.27)
-				)
+		(property "Value" "+3.3V_DP_LORA"
+			(at 112.522 141.478 0)
+			(show_name no)
+			(do_not_autoplace no)
+			(effects
+				(font
+					(size 1.27 1.27)
+				)
+				(justify right)
 			)
 		)
@@
 		(in_pos_files yes)
 		(dnp no)
-		(fields_autoplaced yes)
 		(property "Reference" "#PWR057"
 			(at 179.07 86.36 0)
@@
 			)
 		)
-		(property "Value" "+3.3V_DISP"
-			(at 173.99 90.1699 90)
-			(show_name no)
-			(do_not_autoplace no)
-			(effects
-				(font
-					(size 1.27 1.27)
-				)
-				(justify left)
+		(property "Value" "+3.3V_DP_LORA"
+			(at 172.974 87.63 90)
+			(show_name no)
+			(do_not_autoplace no)
+			(effects
+				(font
+					(size 1.27 1.27)
+				)
 			)
 		)
@@
 			)
 		)
-		(property "Value" "+3.3V"
+		(property "Value" "+3.3V_DP_LORA"
 			(at 112.776 124.46 0)
 			(show_name no)
@@
 				(font
 					(size 0.889 0.889)
-				)
-			)
+					(color 255 0 230 1)
+				)
+			)

Commit message: changed screen footprint
Parts:
- J4: footprint Connector_PinHeader_2.54mm:PinHeader_1x40_P2.54mm_Vertical -> Connector_FFC-FPC:Amphenol_F32Q-1A7x1-11039_1x39-1MP_P0.5mm_Horizontal
Changed lines of the file:
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@@
 			)
 		)
-		(property "Footprint" "Connector_PinHeader_2.54mm:PinHeader_1x40_P2.54mm_Vertical"
+		(property "Footprint" "Connector_FFC-FPC:Amphenol_F32Q-1A7x1-11039_1x39-1MP_P0.5mm_Horizontal"
 			(at 148.59 66.04 0)
 			(hide yes)

Commit message: Updated footprints fixed DRC errors
Parts:
- J4: footprint Connector_FFC-FPC:Amphenol_F32Q-1A7x1-11039_1x39-1MP_P0.5mm_Horizontal -> Connector_FFC-FPC:TE_4-1734839-0_1x40-1MP_P0.5mm_Horizontal
Changed lines of the file:
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@@
 			)
 		)
-		(property "Footprint" "Connector_FFC-FPC:Amphenol_F32Q-1A7x1-11039_1x39-1MP_P0.5mm_Horizontal"
+		(property "Footprint" "Connector_FFC-FPC:TE_4-1734839-0_1x40-1MP_P0.5mm_Horizontal"
 			(at 148.59 66.04 0)
 			(hide yes)

Commit message: Updated with new power rails, added sensors and gps symbol
Parts:
- C25, C26: value 0.1u -> 100n
Connections:
- net +3.3V_DP_LORA renamed +1.8V
- net +1.8V: no longer J4.33 (Pin_33)
- new net +3.3V_HP: J4.33 (Pin_33)
Other:
- moved on the sheet: C26
Changed lines of the file:
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@@
+	)
+	(junction
+		(at 186.69 72.39)
+		(diameter 0)
+		(color 0 0 0 0)
+	)
+	(junction
+		(at 191.77 74.93)
+		(diameter 0)
+		(color 0 0 0 0)
+	)
+	(junction
+		(at 185.42 72.39)
+		(diameter 0)
+		(color 0 0 0 0)
+	)
+	(junction
+		(at 180.34 96.52)
+		(diameter 0)
+		(color 0 0 0 0)
+	)
+	(junction
+		(at 123.19 124.46)
+		(diameter 0)
+		(color 0 0 0 0)
+	)
+	(junction
+		(at 194.31 74.93)
+		(diameter 0)
+		(color 0 0 0 0)
+	)
+	(junction
+		(at 113.03 85.09)
+		(diameter 0)
+		(color 0 0 0 0)
+	)
+	(junction
+		(at 113.03 105.41)
+		(diameter 0)
+		(color 0 0 0 0)
 	)
 	(junction
@@
 	)
 	(junction
-		(at 186.69 72.39)
-		(diameter 0)
-		(color 0 0 0 0)
-	)
-	(junction
-		(at 191.77 74.93)
-		(diameter 0)
-		(color 0 0 0 0)
-	)
-	(junction
-		(at 185.42 72.39)
-		(diameter 0)
-		(color 0 0 0 0)
-	)
-	(junction
-		(at 180.34 96.52)
-		(diameter 0)
-		(color 0 0 0 0)
-	)
-	(junction
-		(at 123.19 124.46)
-		(diameter 0)
-		(color 0 0 0 0)
-	)
-	(junction
-		(at 194.31 74.93)
-		(diameter 0)
-		(color 0 0 0 0)
-	)
-	(junction
-		(at 113.03 85.09)
-		(diameter 0)
-		(color 0 0 0 0)
-	)
-	(junction
-		(at 113.03 105.41)
-		(diameter 0)
-		(color 0 0 0 0)
-	)
-	(junction
 		(at 113.03 95.25)
 		(diameter 0)
@@
 	(wire
 		(pts
-			(xy 104.14 127) (xy 110.49 127)
+			(xy 100.33 127) (xy 110.49 127)
 		)
 		(stroke
@@
 	(wire
 		(pts
-			(xy 104.14 120.65) (xy 104.14 127)
+			(xy 100.33 120.65) (xy 100.33 127)
 		)
 		(stroke
@@
 	(wire
 		(pts
-			(xy 111.76 120.65) (xy 113.03 120.65)
+			(xy 107.95 120.65) (xy 113.03 120.65)
 		)
 		(stroke
@@
 			)
 		)
-		(property "Value" "+3.3V_DP_LORA"
-			(at 202.184 80.518 0)
+		(property "Value" "+1.8V"
+			(at 196.85 80.772 0)
 			(show_name no)
 			(do_not_autoplace no)
@@
 			)
 		)
-		(property "Value" "+3.3V_DP_LORA"
+		(property "Value" "+1.8V"
 			(at 112.522 141.478 0)
 			(show_name no)
@@
 			)
 		)
-		(property "Value" "0.1u"
+		(property "Value" "100n"
 			(at 119.38 132.08 90)
 			(show_name no)
@@
 			)
 		)
-		(property "Value" "+3.3V_DP_LORA"
-			(at 172.974 87.63 90)
+		(property "Value" "+3.3V_HP"
+			(at 169.926 90.17 90)
 			(show_name no)
 			(do_not_autoplace no)
@@
 	(symbol
 		(lib_id "Device:C")
-		(at 107.95 120.65 90)
+		(at 104.14 120.65 90)
 		(unit 1)
 		(body_style 1)
@@
 		(fields_autoplaced yes)
 		(property "Reference" "C26"
-			(at 107.95 113.03 90)
-			(show_name no)
-			(do_not_autoplace no)
-			(effects
-				(font
-					(size 1.27 1.27)
-				)
-			)
-		)
-		(property "Value" "0.1u"
-			(at 107.95 115.57 90)
+			(at 104.14 113.03 90)
+			(show_name no)
+			(do_not_autoplace no)
+			(effects
+				(font
+					(size 1.27 1.27)
+				)
+			)
+		)
+		(property "Value" "100n"
+			(at 104.14 115.57 90)
 			(show_name no)
 			(do_not_autoplace no)
@@
 		)
 		(property "Footprint" "Capacitor_SMD:C_0603_1608Metric"
-			(at 111.76 119.6848 0)
+			(at 107.95 119.6848 0)
 			(hide yes)
 			(show_name no)
@@
 		)
 		(property "Datasheet" ""
-			(at 107.95 120.65 0)
+			(at 104.14 120.65 0)
 			(hide yes)
 			(show_name no)
@@
 		)
 		(property "Description" "Unpolarized capacitor"
-			(at 107.95 120.65 0)
+			(at 104.14 120.65 0)
 			(hide yes)
 			(show_name no)
@@
 		)
 		(property "KLC_S3.3" ""
-			(at 107.95 120.65 90)
+			(at 104.14 120.65 90)
 			(hide yes)
 			(show_name no)
@@
 		)
 		(property "KLC_S4.1" ""
-			(at 107.95 120.65 90)
+			(at 104.14 120.65 90)
 			(hide yes)
 			(show_name no)
@@
 			)
 		)
-		(property "Value" "+3.3V_DP_LORA"
+		(property "Value" "+1.8V"
 			(at 112.776 124.46 0)
 			(show_name no)
@@
 				(font
 					(size 0.889 0.889)
-					(color 255 0 230 1)
-				)
-			)
+				)
+			)

Commit message: added mux for usb, cleaned up schematic for pcb design, setup new pcb with correct size
Other:
- note added: "Screen Connector"
- moved on the sheet: C25, C26, C27, J4, Q1, R10, R11, R6, R7, R8, R9

Commit message: pcb draft, cleaned up schematic
Connections:
- net +1.8V: now also J4.38 (Pin_38)
- net GND: no longer J4.38 (Pin_38)
- net LCD_D10: no longer names the net of J4.27 (Pin_27)
- net LCD_D11: no longer names the net of J4.28 (Pin_28)
- net LCD_D12: no longer names the net of J4.29 (Pin_29)
- net LCD_D13: no longer names the net of J4.30 (Pin_30)
- net LCD_D14: no longer names the net of J4.31 (Pin_31)
- net LCD_D15: no longer names the net of J4.32 (Pin_32)
- net LCD_D8: no longer names the net of J4.25 (Pin_25)
- net LCD_D9: no longer names the net of J4.26 (Pin_26)
- no-connect marks 3 -> 11
Changed lines of the file:
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@@
-	)
-	(junction
-		(at 190.5 71.12)
-		(diameter 0)
-		(color 0 0 0 0)
 	)
 	(junction
@@
 	)
 	(junction
+		(at 195.58 72.39)
+		(diameter 0)
+		(color 0 0 0 0)
+	)
+	(junction
 		(at 179.07 92.71)
 		(diameter 0)
@@
 	)
 	(junction
+		(at 190.5 69.85)
+		(diameter 0)
+		(color 0 0 0 0)
+	)
+	(junction
 		(at 121.92 120.65)
 		(diameter 0)
@@
 	)
 	(junction
-		(at 193.04 71.12)
-		(diameter 0)
-		(color 0 0 0 0)
-	)
-	(junction
 		(at 111.76 81.28)
 		(diameter 0)
@@
 	)
 	(no_connect
+		(at 167.64 67.31)
+	)
+	(no_connect
+		(at 172.72 67.31)
+	)
+	(no_connect
 		(at 129.54 67.31)
 	)
 	(no_connect
+		(at 160.02 67.31)
+	)
+	(no_connect
+		(at 170.18 67.31)
+	)
+	(no_connect
+		(at 177.8 67.31)
+	)
+	(no_connect
 		(at 132.08 67.31)
 	)
@@
 		(at 116.84 67.31)
 	)
+	(no_connect
+		(at 162.56 67.31)
+	)
+	(no_connect
+		(at 175.26 67.31)
+	)
+	(no_connect
+		(at 165.1 67.31)
+	)
 	(wire
 		(pts
@@
 	(wire
 		(pts
-			(xy 193.04 71.12) (xy 193.04 67.31)
-		)
-		(stroke
-			(width 0)
-			(type default)
-		)
-	)
-	(wire
-		(pts
 			(xy 106.68 67.31) (xy 106.68 69.85)
 		)
@@
 	(wire
 		(pts
+			(xy 195.58 67.31) (xy 195.58 72.39)
+		)
+		(stroke
+			(width 0)
+			(type default)
+		)
+	)
+	(wire
+		(pts
 			(xy 137.16 67.31) (xy 137.16 80.01)
 		)
@@
 	(wire
 		(pts
-			(xy 190.5 71.12) (xy 193.04 71.12)
-		)
-		(stroke
-			(width 0)
-			(type default)
-		)
-	)
-	(wire
-		(pts
 			(xy 189.23 85.09) (xy 189.23 87.63)
 		)
@@
 	(wire
 		(pts
+			(xy 198.12 69.85) (xy 190.5 69.85)
+		)
+		(stroke
+			(width 0)
+			(type default)
+		)
+	)
+	(wire
+		(pts
 			(xy 99.06 67.31) (xy 99.06 81.28)
 		)
@@
 	(wire
 		(pts
-			(xy 198.12 67.31) (xy 198.12 71.12)
-		)
-		(stroke
-			(width 0)
-			(type default)
-		)
-	)
-	(wire
-		(pts
-			(xy 195.58 67.31) (xy 195.58 72.39)
-		)
-		(stroke
-			(width 0)
-			(type default)
-		)
-	)
-	(wire
-		(pts
 			(xy 121.92 102.87) (xy 121.92 120.65)
 		)
@@
 	(wire
 		(pts
+			(xy 198.12 67.31) (xy 198.12 69.85)
+		)
+		(stroke
+			(width 0)
+			(type default)
+		)
+	)
+	(wire
+		(pts
 			(xy 93.98 69.85) (xy 93.98 101.6)
 		)
@@
 	(wire
 		(pts
+			(xy 193.04 72.39) (xy 195.58 72.39)
+		)
+		(stroke
+			(width 0)
+			(type default)
+		)
+	)
+	(wire
+		(pts
 			(xy 180.34 86.36) (xy 176.53 86.36)
 		)
@@
 	(wire
 		(pts
-			(xy 190.5 67.31) (xy 190.5 71.12)
-		)
-		(stroke
-			(width 0)
-			(type default)
-		)
-	)
-	(wire
-		(pts
 			(xy 109.22 102.87) (xy 109.22 123.19)
 		)
@@
 	(wire
 		(pts
-			(xy 198.12 71.12) (xy 193.04 71.12)
-		)
-		(stroke
-			(width 0)
-			(type default)
-		)
-	)
-	(wire
-		(pts
 			(xy 179.07 102.87) (xy 189.23 102.87)
 		)
@@
 	(wire
 		(pts
-			(xy 190.5 71.12) (xy 190.5 72.39)
+			(xy 190.5 69.85) (xy 190.5 72.39)
+		)
+		(stroke
+			(width 0)
+			(type default)
+		)
+	)
+	(wire
+		(pts
+			(xy 190.5 67.31) (xy 190.5 69.85)
+		)
+		(stroke
+			(width 0)
+			(type default)
+		)
+	)
+	(wire
+		(pts
+			(xy 193.04 67.31) (xy 193.04 72.39)
 		)
 		(stroke
@@
 		)
 	)
-	(global_label "LCD_D12"
-		(shape input)
-		(at 170.18 67.31 270)
-		(fields_autoplaced yes)
-		(effects
-			(font
-				(size 1.27 1.27)
-			)
-			(justify right)
-		)
-		(property "Intersheetrefs" "${INTERSHEET_REFS}"
-			(at 170.18 77.3104 90)
-			(hide yes)
-			(show_name no)
-			(do_not_autoplace no)
-			(effects
-				(font
-					(size 1.27 1.27)
-				)
-				(justify right)
-			)
-		)
-	)
 	(global_label "LCD_NE1"
 		(shape input)
@@
 		)
 	)
-	(global_label "LCD_D15"
-		(shape input)
-		(at 177.8 67.31 270)
-		(fields_autoplaced yes)
-		(effects
-			(font
-				(size 1.27 1.27)
-			)
-			(justify right)
-		)
-		(property "Intersheetrefs" "${INTERSHEET_REFS}"
-			(at 177.8 77.3104 90)
-			(hide yes)
-			(show_name no)
-			(do_not_autoplace no)
-			(effects
-				(font
-					(size 1.27 1.27)
-				)
-				(justify right)
-			)
-		)
-	)
 	(global_label "CTP_INT"
 		(shape input)
@@
 		)
 	)
-	(global_label "LCD_D10"
-		(shape input)
-		(at 165.1 67.31 270)
-		(fields_autoplaced yes)
-		(effects
-			(font
-				(size 1.27 1.27)
-			)
-			(justify right)
-		)
-		(property "Intersheetrefs" "${INTERSHEET_REFS}"
-			(at 165.1 77.3104 90)
-			(hide yes)
-			(show_name no)
-			(do_not_autoplace no)
-			(effects
-				(font
-					(size 1.27 1.27)
-				)
-				(justify right)
-			)
-		)
-	)
 	(global_label "LCD_D7"
 		(shape input)
@@
 		)
 	)
-	(global_label "LCD_D11"
-		(shape input)
-		(at 167.64 67.31 270)
-		(fields_autoplaced yes)
-		(effects
-			(font
-				(size 1.27 1.27)
-			)
-			(justify right)
-		)
-		(property "Intersheetrefs" "${INTERSHEET_REFS}"
-			(at 167.64 77.3104 90)
-			(hide yes)
-			(show_name no)
-			(do_not_autoplace no)
-			(effects
-				(font
-					(size 1.27 1.27)
-				)
-				(justify right)
-			)
-		)
-	)
 	(global_label "CTP_SCL"
 		(shape input)
@@
 		)
 	)
-	(global_label "LCD_D13"
-		(shape input)
-		(at 172.72 67.31 270)
-		(fields_autoplaced yes)
-		(effects
-			(font
-				(size 1.27 1.27)
-			)
-			(justify right)
-		)
-		(property "Intersheetrefs" "${INTERSHEET_REFS}"
-			(at 172.72 77.3104 90)
-			(hide yes)
-			(show_name no)
-			(do_not_autoplace no)
-			(effects
-				(font
-					(size 1.27 1.27)
-				)
-				(justify right)
-			)
-		)
-	)
 	(global_label "LCD_D0"
 		(shape input)
@@
 		)
 	)
-	(global_label "LCD_D9"
-		(shape input)
-		(at 162.56 67.31 270)
-		(fields_autoplaced yes)
-		(effects
-			(font
-				(size 1.27 1.27)
-			)
-			(justify right)
-		)
-		(property "Intersheetrefs" "${INTERSHEET_REFS}"
-			(at 162.56 77.3104 90)
-			(hide yes)
-			(show_name no)
-			(do_not_autoplace no)
-			(effects
-				(font
-					(size 1.27 1.27)
-				)
-				(justify right)
-			)
-		)
-	)
 	(global_label "LCD_D2"
 		(shape input)
@@
 		)
 	)
-	(global_label "LCD_D14"
-		(shape input)
-		(at 175.26 67.31 270)
-		(fields_autoplaced yes)
-		(effects
-			(font
-				(size 1.27 1.27)
-			)
-			(justify right)
-		)
-		(property "Intersheetrefs" "${INTERSHEET_REFS}"
-			(at 175.26 77.3104 90)
-			(hide yes)
-			(show_name no)
-			(do_not_autoplace no)
-			(effects
-				(font
-					(size 1.27 1.27)
-				)
-				(justify right)
-			)
-		)
-	)
 	(global_label "LCD_RS"
 		(shape input)
@@
 			(hide yes)
 			(show_name no)
-			(do_not_autoplace no)
-			(effects
-				(font
-					(size 1.27 1.27)
-				)
-				(justify right)
-			)
-		)
-	)
-	(global_label "LCD_D8"
-		(shape input)
-		(at 160.02 67.31 270)
-		(fields_autoplaced yes)
-		(effects
-			(font
-				(size 1.27 1.27)
-			)
-			(justify right)
-		)
-		(property "Intersheetrefs" "${INTERSHEET_REFS}"
-			(at 160.02 77.3104 90)
-			(hide yes)
-			(show_name no)
