File: TheSummitProject.kicad_pcb (KiCad board)
At the start: 2 copper layers, 53 x 80 mm, 104 parts, among them IC1 STM32U5F7VJT6, J1 Cortex SWD, J2 GPS_ANT, J4 Screen FPC, J5 Micro_SD_Card_Det1, Q1 NMOS, Q2 PMOS, SW1 SW_SPDT, SW2 PWR_BTN, U1 NPM1300-CAAA-R, U10 TS3USB30EDGSR, U2 USBLC6-2SC6, U3 USBLC6-2SC6, U4 TPS62840DLCR, U5 BME280, U6 LSM303AGR, U7 MAX-M10S-00B, U8 RAK4630, U9 SN74AVC2T245RSWR, Y1 16Mhz, Y2 32.768Khz

Commit message: Changed SPI to 3-wire, added Accelerometer interupt
Connections:
- IC1 pad 90: SNSR_MISO -> ACC_INT
- U5 pad 5: SNSR_MISO -> unconnected-(U5-SDO-Pad5)
- U6 pad 12: unconnected-(U6-INT_1_XL-Pad12) -> ACC_INT
- U7 pad 2: GPS_TX -> GPS_RX
- U7 pad 3: GPS_RX -> GPS_TX
Changed lines of the file:
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@@
 			(size 0.5 0.35)
 			(layers "F.Cu" "F.Mask" "F.Paste")
-			(net "SNSR_MISO")
+			(net "unconnected-(U5-SDO-Pad5)")
 			(pinfunction "SDO_5")
-			(pintype "bidirectional")
+			(pintype "bidirectional+no_connect")
 		)
 		(pad "6" smd rect
@@
 			(layers "F.Cu" "F.Mask" "F.Paste")
 			(net "GPS_INT")
-			(pinfunction "PC2_17")
+			(pinfunction "GPS_INT_17")
 			(pintype "passive")
 		)
@@
 			(size 0.3 1.475)
 			(layers "F.Cu" "F.Mask" "F.Paste")
-			(net "SNSR_MISO")
-			(pinfunction "SNSR_MISO_90")
+			(net "ACC_INT")
+			(pinfunction "ACC_INT_90")
 			(pintype "passive")
 		)
@@
 			(size 0.35 0.43)
 			(layers "F.Cu" "F.Mask" "F.Paste")
-			(net "unconnected-(U6-INT_1_XL-Pad12)")
+			(net "ACC_INT")
 			(pinfunction "INT_1_XL_12")
-			(pintype "output+no_connect")
+			(pintype "output")
 			(solder_mask_margin 0.102)
 		)
@@
 			(size 1.8 0.8)
 			(layers "F.Cu" "F.Mask")
-			(net "GPS_TX")
+			(net "GPS_RX")
 			(pinfunction "TXD_2")
 			(pintype "output")
@@
 			(size 1.8 0.8)
 			(layers "F.Cu" "F.Mask")
-			(net "GPS_RX")
+			(net "GPS_TX")
 			(pinfunction "RXD_3")
 			(pintype "input")

Commit message: pcb v2 layer change placed chip
Parts:
- C6: moved to B.Cu
- moved C7 156.4 mm to (211.3, 73.5)
- moved Q1 145.0 mm to (185.8, 40.9)
- moved Q2 145.0 mm to (185.8, 45.4)
- moved U2 145.0 mm to (180.8, 41.1)
- moved U3 141.9 mm to (178.9, 48.5)
- moved U10 134.8 mm to (193.3, 64.5)
- moved USB-C1 113.7 mm to (170.0, 83.0), turned to 90 degrees
- moved C3 106.9 mm to (153.5, 113.0), turned to -90 degrees
- moved C2 106.6 mm to (158.5, 94.5)
- moved C8 103.3 mm to (158.5, 92.5)
- moved U6 98.6 mm to (145.8, 83.8)
- moved U4 97.4 mm to (157.7, 123.2)
- moved J4 96.6 mm to (160.8, 134.8)
- moved C4 95.3 mm to (142.0, 113.0), turned to -90 degrees
- moved U1 93.9 mm to (165.0, 122.0)
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Routing:
- net GND: track 0.00 -> 26.0 mm, vias 0 -> 18
- net +1.8V: track 0.00 -> 21.0 mm
- net Net-(IC1-HSE_IN): track 0.00 -> 12.0 mm
- net Net-(IC1-HSE_OUT): track 0.00 -> 9.71 mm
- net Net-(IC1-LSE_IN): track 0.00 -> 7.17 mm
- net Net-(IC1-LSE_OUT): track 0.00 -> 6.69 mm
- added copper zone on In1.Cu, net GND
Other:
- copper layers 2 -> 4

Commit message: pcb draft, cleaned up schematic
Parts:
- removed C10, C11, C18: 1u, Capacitor_SMD:C_0603_1608Metric
- removed C6, C7: 100n, Capacitor_SMD:C_0603_1608Metric
- removed FB1: 120R, Inductor_SMD:L_0603_1608Metric
- added BZ1: PKLCS1212E4001-R1, Buzzer_Beeper:Buzzer_Murata_PKLCS1212E, F.Cu at (79.7, 57.8)
- added R29: 100, Resistor_SMD:R_0603_1608Metric, F.Cu at (66.5, 90.3)
- C1, C19, C2, C3, C4, C5, C8, C9, U8: moved to B.Cu
- moved U6 97.7 mm to (77.4, 153.5)
- moved C9 96.4 mm to (142.8, 87.8)
- moved C19 95.6 mm to (145.8, 87.8)
- moved U9 71.7 mm to (73.4, 153.7)
- moved BATT1 63.6 mm to (205.0, 114.9)
- moved U8 55.8 mm to (147.8, 124.5), turned to 180 degrees
- moved C4 40.8 mm to (147.0, 72.5), turned to 0 degrees
- moved J2 39.8 mm to (83.5, 103.5)
- moved U4 39.5 mm to (194.7, 137.0)
- moved U5 39.5 mm to (185.0, 130.2)
- moved J4 37.4 mm to (147.2, 100.0)
- moved C3 34.3 mm to (154.2, 78.8), turned to 180 degrees
- moved J5 28.1 mm to (103.8, 137.0)
- moved IC1 21.5 mm to (147.0, 79.5), turned to 45 degrees
- moved U7 19.1 mm to (111.0, 79.5)
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Connections:
- C19 pad 1: +1.8VA -> +1.8V
- C9 pad 1: +1.8VA -> GND
- C9 pad 2: GND -> +1.8V
- IC1 pad 2: unconnected-(IC1-PE3-Pad2) -> PIEZO_P1
- IC1 pad 21: +1.8VA -> +1.8V
- IC1 pad 22: +1.8VA -> +1.8V
- IC1 pad 3: unconnected-(IC1-PE4-Pad3) -> PIEZO_P2
- IC1 pad 42: LCD_D8 -> unconnected-(IC1-LCD_D8-Pad42)
- IC1 pad 43: LCD_D9 -> unconnected-(IC1-LCD_D9-Pad43)
- IC1 pad 44: LCD_D10 -> unconnected-(IC1-LCD_D10-Pad44)
- IC1 pad 45: LCD_D11 -> unconnected-(IC1-LCD_D11-Pad45)
- IC1 pad 46: LCD_D12 -> unconnected-(IC1-LCD_D12-Pad46)
- IC1 pad 55: LCD_D13 -> unconnected-(IC1-LCD_D13-Pad55)
- IC1 pad 56: LCD_D14 -> unconnected-(IC1-LCD_D14-Pad56)
- IC1 pad 57: LCD_D15 -> unconnected-(IC1-LCD_D15-Pad57)
- J4 pad 25: LCD_D8 -> unconnected-(J4-Pin_25-Pad25)
- J4 pad 26: LCD_D9 -> unconnected-(J4-Pin_26-Pad26)
- J4 pad 27: LCD_D10 -> unconnected-(J4-Pin_27-Pad27)
- J4 pad 28: LCD_D11 -> unconnected-(J4-Pin_28-Pad28)
- J4 pad 29: LCD_D12 -> unconnected-(J4-Pin_29-Pad29)
- J4 pad 30: LCD_D13 -> unconnected-(J4-Pin_30-Pad30)
- J4 pad 31: LCD_D14 -> unconnected-(J4-Pin_31-Pad31)
- J4 pad 32: LCD_D15 -> unconnected-(J4-Pin_32-Pad32)
- J4 pad 38: GND -> +1.8V
Routing:
- net GND: track 26.0 -> 83.8 mm, vias 18 -> 26
- net Net-(IC1-LSE_OUT): track 6.69 -> 13.0 mm
- net Net-(IC1-LSE_IN): track 7.17 -> 11.5 mm
- net +1.8V: track 21.0 -> 23.1 mm, vias 0 -> 11
- net Net-(IC1-HSE_OUT): track 9.71 -> 11.7 mm

Commit message: PCB DRAFT
Parts:
- C12, C13, C25, C26, C27, R1, R7, R8: moved to B.Cu
- moved C12 106.8 mm to (151.8, 80.3), turned to -45 degrees
- moved R10 106.6 mm to (165.5, 95.0)
- moved R11 106.6 mm to (165.5, 97.5)
- moved C13 97.6 mm to (143.5, 83.0)
- moved C25 89.8 mm to (140.0, 93.8), turned to 90 degrees
- moved C26 87.6 mm to (137.8, 97.0)
- moved C27 87.3 mm to (137.7, 95.5), turned to 180 degrees
- moved U1 77.3 mm to (159.5, 45.5)
- moved R6 75.0 mm to (132.3, 98.0), turned to 180 degrees
- moved R8 73.0 mm to (131.2, 96.5), turned to 180 degrees
- moved R7 71.4 mm to (129.5, 95.0), turned to 180 degrees
- moved R1 71.1 mm to (129.5, 72.0)
- moved Q1 58.6 mm to (159.0, 93.0)
- moved J1 50.4 mm to (144.5, 63.5), turned to 90 degrees
- moved SW1 35.3 mm to (127.5, 66.5), turned to 180 degrees
Routing:
- net CTP_SCL: track 0.00 -> 50.2 mm
- net CTP_INT: track 0.00 -> 49.6 mm, vias 0 -> 3
- net CTP_SDA: track 0.00 -> 45.1 mm, vias 0 -> 1
- net CTP_RST: track 0.00 -> 44.4 mm, vias 0 -> 2
- net LCD_NE1: track 0.00 -> 39.9 mm, vias 0 -> 4
- net LCD_NOE: track 0.00 -> 37.9 mm, vias 0 -> 2
- net LCD_NWE: track 0.00 -> 36.1 mm, vias 0 -> 3
- net LCD_RST: track 0.00 -> 35.9 mm, vias 0 -> 2
- net /MCU/NRST: track 0.00 -> 31.6 mm, vias 0 -> 3
- net +1.8V: track 23.1 -> 41.7 mm, vias 11 -> 19
- net LCD_D7: track 0.00 -> 17.6 mm
- net LCD_D6: track 0.00 -> 17.3 mm
- net GND: track 83.8 -> 100.8 mm, vias 26 -> 39
- net LCD_D5: track 0.00 -> 16.9 mm
- net LCD_D4: track 0.00 -> 16.6 mm
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